File: Hardware/ADS124S08-Dev-Board/ADS124S08-Dev-Board.brd (EAGLE design)
At the start: 33 x 20.3 mm, 12 parts, among them U1 ADS124S08IPBSR

Commit message: Component placement done
Parts:
- added FB1: (no value), electroShri:_0603
- added GOLD_ORB_SM1: OSHWLOGOLOGO5MM, electroShri:OSHW_5MM
- added GOLD_ORB_SM2: OSHWLOGOLOGO8MM, electroShri:OSHW_8MM
- moved C1 9.31 mm to (6.25, 15.2), turned to 90 degrees
- moved C5 7.02 mm to (12.0, 11.5)
- moved C3 1.22 mm to (12.0, 4.50)
- moved R1 0.50 mm to (8.50, 15.2)
- moved R2 0.50 mm to (10.5, 15.2)
- moved R3 0.50 mm to (12.5, 15.2)
- moved R4 0.50 mm to (14.5, 15.2)
- moved R5 0.50 mm to (16.5, 15.2)
- moved R6 0.50 mm to (18.5, 15.2)
- moved R7 0.50 mm to (20.5, 15.2)
Connections:
- net AGND: now also FB1.1
- net DGND: now also FB1.2
Routing:
- net AGND: track 0.00 -> 39.5 mm, vias 0 -> 6
- net +5V: track 0.00 -> 28.0 mm, vias 0 -> 1
- net DGND: track 0.00 -> 19.8 mm, vias 0 -> 2
- net AIN11: track 0.00 -> 18.8 mm
- net REFP0: track 0.00 -> 18.1 mm, vias 0 -> 1
- net REFN0: track 0.00 -> 17.3 mm, vias 0 -> 1
- net 3V3: track 0.00 -> 16.8 mm, vias 0 -> 1
- net AIN0: track 0.00 -> 16.8 mm
- net AIN10: track 0.00 -> 15.7 mm
- net N$7: track 0.00 -> 15.6 mm, vias 0 -> 2
- net AIN1: track 0.00 -> 15.0 mm
- net AIN2: track 0.00 -> 13.1 mm
- net AIN9: track 0.00 -> 12.9 mm
- net AIN3: track 0.00 -> 11.4 mm
- net AIN4: track 0.00 -> 10.6 mm
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Other:
- board text added: "+5V"
- board text added: "3V3"
- board text added: "A0"
- board text added: "A1"
- board text added: "A10"
- board text added: "A11"
- board text added: "A2"
- board text added: "A3"
- board text added: "A4"
- board text added: "A5"
- board text added: "A6"
- board text added: "A7"
- board text added: "A8"
- board text added: "A9"
- board text added: "ADS124S08 delta-sigma ADC 24-bit, 4-kSPS, 12-ch"
- board text added: "AGND"
- board text added: "CLK"
- board text added: "CS"
- board text added: "DRDY"
- board text added: "GND"
- board text added: "MISO"
- board text added: "MOSI"
- board text added: "REFN"
- board text added: "REFP"
- board text added: "RST"
- board text added: "STRT"
- board text added: "https:// shridattdudhat.github.io/ ADS124S08"
- board text added: "https://shridattdudhat.github.io/"
