File: Hardware/ADS124S08-Dev-Board/ADS124S08-Dev-Board.sch (EAGLE design)
At the start: 12 parts, among them U1 ADS124S08IPBSR

Commit message: Component placement done
Parts:
- added FB1: (no value), electroShri:FERRITE_0603
- added GOLD_ORB_SM1: OSHWLOGOLOGO5MM, electroShri:OSHWLOGOLOGO5MM
- added GOLD_ORB_SM2: OSHWLOGOLOGO8MM, electroShri:OSHWLOGOLOGO8MM
Connections:
- net AGND: now also FB1.P$1
- net DGND: now also FB1.P$2
